File: hardware/myco-mini-host-pcb/myco-mini-host-pcb.kicad_sch (KiCad schematic)
At the start: 37 parts, among them J1 Conn_01x17_Female, J2 Conn_01x17_Female, Q1 AO3401A, Q2 AO3401A, Q3 AO3401A, Q4 AO3401A, SW1 DM-04-V, SW2 TS-1187A-B-A-B, U1 XC9145B33CMR-G, U2 SHT41-AD1B-R2, U3 BH1750FVI-TR, U4 MAX40203AUK+T

Commit message: fix: pads thermiques U2/U3 en no-connect, R14 sur ADDR du BH1750
Les deux dernieres decisions de l'audit #2, tranchees par l'utilisateur.

- Pads thermiques U2 (pin5) / U3 (pin7) : l'isolation faite sur le PCB est
  intentionnelle (isolation thermique du SHT41, et Sensirion deconseille de
  souder son pad central). Le schema les reliait encore a GND, donc la
  prochaine synchro "Update PCB from Schematic" les aurait re-relies en
  silence. Remplace par des drapeaux no-connect explicites.

- R14 (100k) entre ADDR du BH1750 et GND. ROHM prescrit une resistance
  (~100k) plutot qu'une liaison directe quand aucune impulsion basse de
  >=1us n'est appliquee sur DVI au demarrage : c'est exactement notre cas,
  DVI etant cablee en dur sur SENSOR_3V3 (elle monte AVEC VCC). Et comme
  SENSOR_3V3 est desormais commute par Q3, cette sequence se rejoue a chaque
  cycle de mesure au lieu d'une seule fois au boot. ADDR reste lue a l'etat
  bas, adresse I2C inchangee (0x23).
  Contrainte de placement : ADDR ne peut pas descendre verticalement, la
  broche GND de U3 est sur le meme axe X - un fil droit les aurait
  court-circuitees, d'ou le coude vers la gauche avant R14.

- Note firmware (P1.10/P1.11 en entree deconnectee quand SENSOR_EN est bas)
  ouverte en issue GitHub #19. Commentaire ajoute sur l'issue #17 pour
  documenter le fix d'orientation de Q1 et signaler que le brief sec.4
  contient toujours l'orientation erronee.

- BOM : R14 ajoutee. Verifie 38 composants schema = 38 BOM.

Alignement des textes preserve : diff UUID avant/apres sur les 79 labels,
zero deplacement. ERC 71 -> 69, DRC 0 violation.

Co-Authored-By: Claude Sonnet 5 <noreply@anthropic.com>
Parts:
- added R14: 100k, Resistor_SMD:R_0603_1608Metric, symbol Device:R
Connections:
- net GND: now also R14.2; no longer U2.5 (EP), U3.2 (ADDR), U3.7 (EP)
- new net: R14.1, U3.2 (ADDR)
- no-connect marks 17 -> 19
Changed lines of the file:
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@@
 		(at 97.79 173.99)
 	)
+	(no_connect
+		(at 119.38 127)
+	)
+	(no_connect
+		(at 187.96 129.54)
+	)
 	(wire
 		(pts
@@
 	(wire
 		(pts
-			(xy 119.38 127) (xy 134.62 127)
-		)
-		(stroke
-			(width 0)
-			(type default)
-		)
-	)
-	(wire
-		(pts
 			(xy 194.31 204.47) (xy 194.31 208.28)
 		)
@@
 	(wire
 		(pts
-			(xy 187.96 129.54) (xy 214.63 129.54)
-		)
-		(stroke
-			(width 0)
-			(type default)
-		)
-	)
-	(wire
-		(pts
 			(xy 185.42 73.66) (xy 185.42 69.85)
 		)
@@
 		)
 	)
+	(wire
+		(pts
+			(xy 152.4 134.62) (xy 144.78 134.62)
+		)
+		(stroke
+			(width 0)
+			(type default)
+		)
+	)
+	(wire
+		(pts
+			(xy 144.78 134.62) (xy 144.78 143.51)
+		)
+		(stroke
+			(width 0)
+			(type default)
+		)
+	)
+	(wire
+		(pts
+			(xy 144.78 151.13) (xy 144.78 154.94)
+		)
+		(stroke
+			(width 0)
+			(type default)
+		)
+	)
 	(label "SENSOR_3V3"
 		(at 129.54 92.71 0)
@@
 	(symbol
 		(lib_id "power:GND")
-		(at 152.4 134.62 0)
-		(unit 1)
-		(body_style 1)
-		(exclude_from_sim no)
-		(in_bom yes)
-		(on_board yes)
-		(in_pos_files yes)
-		(dnp no)
-		(property "Reference" "#PWR15"
-			(at 152.4 140.62 0)
-			(hide yes)
-			(show_name no)
-			(do_not_autoplace no)
-			(effects
-				(font
-					(size 1.27 1.27)
-				)
-			)
-		)
-		(property "Value" "GND"
-			(at 152.4 138.62 0)
-			(show_name no)
-			(do_not_autoplace no)
-			(effects
-				(font
-					(size 1.27 1.27)
-				)
-			)
-		)
-		(property "Footprint" ""
-			(at 152.4 134.62 0)
-			(hide yes)
-			(show_name no)
-			(do_not_autoplace no)
-			(effects
-				(font
-					(size 1.27 1.27)
-				)
-			)
-		)
-		(property "Datasheet" ""
-			(at 152.4 134.62 0)
-			(show_name no)
-			(do_not_autoplace no)
-			(effects
-				(font
-					(size 1.27 1.27)
-				)
-			)
-		)
-		(property "Description" ""
-			(at 152.4 134.62 0)
-			(show_name no)
-			(do_not_autoplace no)
-			(effects
-				(font
-					(size 1.27 1.27)
-				)
-			)
-		)
-		(pin "1"
-		)
-		(instances
-			(project "myco-mini-host-pcb"
-				(path "/b1969cb4-f84b-4d7e-8508-ab863aa656b2"
-					(reference "#PWR15")
-					(unit 1)
-				)
-			)
-		)
-	)
-	(symbol
-		(lib_id "power:GND")
 		(at 416.56 200.66 0)
 		(unit 1)
@@
 	)
 	(symbol
-		(lib_id "power:GND")
-		(at 214.63 129.54 0)
-		(unit 1)
-		(body_style 1)
-		(exclude_from_sim no)
-		(in_bom yes)
-		(on_board yes)
-		(in_pos_files yes)
-		(dnp no)
-		(property "Reference" "#PWR17"
-			(at 214.63 135.54 0)
-			(hide yes)
-			(show_name no)
-			(do_not_autoplace no)
-			(effects
-				(font
-					(size 1.27 1.27)
-				)
-			)
-		)
-		(property "Value" "GND"
-			(at 214.63 133.54 0)
-			(show_name no)
-			(do_not_autoplace no)
-			(effects
-				(font
-					(size 1.27 1.27)
-				)
-			)
-		)
-		(property "Footprint" ""
-			(at 214.63 129.54 0)
-			(hide yes)
-			(show_name no)
-			(do_not_autoplace no)
-			(effects
-				(font
-					(size 1.27 1.27)
-				)
-			)
-		)
-		(property "Datasheet" ""
-			(at 214.63 129.54 0)
-			(show_name no)
-			(do_not_autoplace no)
-			(effects
-				(font
-					(size 1.27 1.27)
-				)
-			)
-		)
-		(property "Description" ""
-			(at 214.63 129.54 0)
-			(show_name no)
-			(do_not_autoplace no)
-			(effects
-				(font
-					(size 1.27 1.27)
-				)
-			)
-		)
-		(pin "1"
-		)
-		(instances
-			(project "myco-mini-host-pcb"
-				(path "/b1969cb4-f84b-4d7e-8508-ab863aa656b2"
-					(reference "#PWR17")
-					(unit 1)
-				)
-			)
-		)
-	)
-	(symbol
 		(lib_id "myco_host:AO3401A")
 		(at 175.26 44.45 0)
@@
 	)
 	(symbol
-		(lib_id "power:GND")
-		(at 134.62 127 0)
-		(unit 1)
-		(body_style 1)
-		(exclude_from_sim no)
-		(in_bom yes)
-		(on_board yes)
-		(in_pos_files yes)
-		(dnp no)
-		(property "Reference" "#PWR14"
-			(at 134.62 133 0)
-			(hide yes)
-			(show_name no)
-			(do_not_autoplace no)
-			(effects
-				(font
-					(size 1.27 1.27)
-				)
-			)
-		)
-		(property "Value" "GND"
-			(at 134.62 131 0)
-			(show_name no)
-			(do_not_autoplace no)
-			(effects
-				(font
-					(size 1.27 1.27)
-				)
-			)
-		)
-		(property "Footprint" ""
-			(at 134.62 127 0)
-			(hide yes)
-			(show_name no)
-			(do_not_autoplace no)
-			(effects
-				(font
-					(size 1.27 1.27)
-				)
-			)
-		)
-		(property "Datasheet" ""
-			(at 134.62 127 0)
-			(show_name no)
-			(do_not_autoplace no)
-			(effects
-				(font
-					(size 1.27 1.27)
-				)
-			)
-		)
-		(property "Description" ""
-			(at 134.62 127 0)
-			(show_name no)
-			(do_not_autoplace no)
-			(effects
-				(font
-					(size 1.27 1.27)
-				)
-			)
-		)
-		(pin "1"
-		)
-		(instances
-			(project "myco-mini-host-pcb"
-				(path "/b1969cb4-f84b-4d7e-8508-ab863aa656b2"
-					(reference "#PWR14")
-					(unit 1)
-				)
-			)
-		)
-	)
-	(symbol
 		(lib_id "myco_host:AO3401A")
 		(at 330.2 44.45 0)
@@
 					(unit 1)
 				)
+			)
+		)
+	)
+	(symbol
+		(lib_id "Device:R")
+		(at 144.78 147.32 0)
+		(unit 1)
+		(body_style 1)
+		(exclude_from_sim no)
+		(in_bom yes)
+		(on_board yes)
+		(in_pos_files yes)
+		(dnp no)
+		(property "Reference" "R14"
+			(at 149.86 144.78 0)
+			(show_name no)
+			(do_not_autoplace no)
+			(effects
+				(font
+					(size 1.27 1.27)
+				)
+			)
+		)
+		(property "Value" "100k"
+			(at 149.86 149.86 0)
+			(show_name no)
+			(do_not_autoplace no)
+			(effects
+				(font
+					(size 1.27 1.27)
+				)
+			)
+		)
+		(property "Footprint" "Resistor_SMD:R_0603_1608Metric"
+			(at 144.78 147.32 0)
+			(hide yes)
+			(show_name no)
+			(do_not_autoplace no)
+			(effects
+				(font
+					(size 1.27 1.27)
+				)
+			)
+		)
+		(property "Datasheet" ""
+			(at 144.78 147.32 0)
+			(hide yes)
+			(show_name no)
+			(do_not_autoplace no)
+			(effects
+				(font
+					(size 1.27 1.27)
+				)
+			)
+		)
+		(property "Description" ""
+			(at 144.78 147.32 0)
+			(hide yes)
+			(show_name no)
+			(do_not_autoplace no)
+			(effects
+				(font
+					(size 1.27 1.27)
+				)
+			)
+		)
+		(property "Note" "BH1750 ADDR pull-down. ROHM's datasheet warns that ADDR/SDA/SCL are not stable unless DVI is held low for >=1us after VCC rises, and in that case prescribes a resistor (approx 100k) on ADDR instead of a direct tie. DVI is hard-tied to SENSOR_3V3 on this board so it rises WITH VCC and no low pulse is possible - and since SENSOR_3V3 is switched by Q3, that power-up sequence now repeats on every measurement cycle rather than once at boot. ADDR still reads low, so the I2C address stays 0x23."
+			(at 144.78 147.32 0)
+			(hide yes)
+			(show_name no)
+			(do_not_autoplace no)
+			(effects
+				(font
+					(size 1.27 1.27)
+				)
+			)
+		)
+		(pin "1"
+		)
+		(pin "2"
+		)
+		(instances
+			(project "myco-mini-host-pcb"
+				(path "/b1969cb4-f84b-4d7e-8508-ab863aa656b2"
+					(reference "R14")
+					(unit 1)
+				)
+			)
+		)
+	)
+	(symbol
+		(lib_id "power:GND")
+		(at 144.78 154.94 0)
+		(unit 1)
+		(body_style 1)
+		(exclude_from_sim no)
+		(in_bom yes)
+		(on_board yes)
+		(in_pos_files yes)
+		(dnp no)
+		(property "Reference" "#PWR30"
+			(at 144.78 160.94 0)
+			(hide yes)
+			(show_name no)
+			(do_not_autoplace no)
+			(effects
+				(font
+					(size 1.27 1.27)
+				)
+			)
+		)
+		(property "Value" "GND"
+			(at 144.78 158.94 0)
+			(show_name no)
+			(do_not_autoplace no)
+			(effects
+				(font
+					(size 1.27 1.27)
+				)
+			)
+		)
+		(property "Footprint" ""
+			(at 144.78 154.94 0)
+			(hide yes)
+			(show_name no)
+			(do_not_autoplace no)
+			(effects
+				(font
+					(size 1.27 1.27)
+				)
+			)
+		)
+		(property "Datasheet" ""
+			(at 144.78 154.94 0)
+			(hide yes)
+			(show_name no)
+			(do_not_autoplace no)
+			(effects
+				(font
+					(size 1.27 1.27)
+				)
+			)
+		)
+		(property "Description" ""
+			(at 144.78 154.94 0)
+			(hide yes)
+			(show_name no)
+			(do_not_autoplace no)
+			(effects
+				(font
+					(size 1.27 1.27)
+				)
+			)
+		)
+		(pin "1"
+		)
+		(instances
+			(project "myco-mini-host-pcb"
+				(path "/b1969cb4-f84b-4d7e-8508-ab863aa656b2"
+					(reference "#PWR30")
+					(unit 1)
+				)
